Commit message: 添加浮动关节控制节点，更新URDF文件，优化坐标变换节点，新增关节控制节点，调整启动文件以支持GUI

File: my_robot/src/robot_3dros/urdf/single_arm_description_float.urdf (robot description, URDF)
Before this commit: robot single_arm, 9 links, 8 joints
Joints:
- joint world_joint: origin xyz=0 0 0.5 rpy=1.57 0 0 -> xyz=0 0 0.5 rpy=1.5708 0 0
