Commit message: 添加truss机器人URDF描述文件，新增STL模型和相关配置，更新CMakeLists以支持安装，优化关节设置

File: my_robot/src/robot_3dros/urdf/double_arms_description_float.urdf (robot description, URDF)
Before this commit: robot robot_3dros, 16 links, 15 joints
Links:
- added link truss_link, mass 21.7746312239973; collision mesh filename=package://truss/meshes/truss_link.STL; visual mesh filename=package://truss/meshes/truss_link.STL
Joints:
- added joint world_to_truss_link: type fixed, parent world, child truss_link, origin xyz=0.9275 0 0 rpy=1.5708 0 3.1415
- joint world_joint: origin xyz=0 0 0.5 rpy=0 1.5708 0 -> xyz=0 0 0.5 rpy=1.5708 1.5708 0

Commit message: 更新关节角度配置文件，调整浮动基座位置，修改URDF文件中的truss_link位置

File: my_robot/src/robot_3dros/urdf/double_arms_description_float.urdf (robot description, URDF)
Before this commit: robot robot_3dros, 17 links, 16 joints
Joints:
- joint world_to_truss_link: origin xyz=0.9275 0 0 rpy=1.5708 0 3.1415 -> xyz=0.6625 0 0 rpy=1.5708 0 3.1415
